Commit message: feat: add second stick
This commit adds a second stick for which the axis of roation of joint 1
has been switched from the y-axis to the z-axis.

File: gazebo_torque_calculation_bug/stick_description/stick.urdf.xacro (robot description, xacro)
@@ -5,4 +5,5 @@
   <xacro:arg name="rpy" default="0 0 0" />
   <xacro:arg name="rotated" default="false" />
+  <xacro:arg name="robot_name" default="stick" />
   <!--Gazebo requires a joint to a link called "world" for statically mounted robots-->
   <link name="world" />
@@ -10,8 +11,8 @@
     <origin xyz="$(arg xyz)" rpy="$(arg rpy)" />
     <parent link="world" />
-    <child link="stick_link1" />
+    <child link="$(arg robot_name)_link1" />
   </joint>
   <!--Create stick example links-->
-  <link name="stick_link1">
+  <link name="$(arg robot_name)_link1">
     <visual>
       <origin xyz="0 0 0.05" />
@@ -32,5 +33,5 @@
     </inertial>
   </link>
-  <link name="stick_link2">
+  <link name="$(arg robot_name)_link2">
     <visual>
       <origin xyz="0 0 0.05" />
@@ -51,5 +52,5 @@
     </inertial>
   </link>
-  <link name="stick_link3">
+  <link name="$(arg robot_name)_link3">
     <visual>
       <origin xyz="0 0 0.05" />
@@ -73,9 +74,9 @@
   <!--  Problem joint-->
   <xacro:if value="$(arg rotated)">    <!--With rotation-->
-    <joint name="stick_joint1" type="revolute">
+    <joint name="$(arg robot_name)_joint1" type="revolute">
       <safety_controller k_position="100.0" k_velocity="40.0" soft_lower_limit="-2.8973" soft_upper_limit="2.8973"/>
       <origin xyz="0 0 0.1" rpy="${pi/2} -${pi/2} 0" />
-      <parent link="stick_link1"/>
-      <child link="stick_link2"/>
+      <parent link="$(arg robot_name)_link1"/>
+      <child link="$(arg robot_name)_link2"/>
       <axis xyz="0 0 1"/>
       <limit acceleration="15" lower="-2.9671" effort="87" upper="2.9671" velocity="2.5"/>
@@ -84,9 +85,9 @@
   </xacro:if>
   <xacro:unless value="$(arg rotated)">
-    <joint name="stick_joint1" type="revolute">
+    <joint name="$(arg robot_name)_joint1" type="revolute">
       <safety_controller k_position="100.0" k_velocity="40.0" soft_lower_limit="-2.8973" soft_upper_limit="2.8973"/>
       <origin xyz="0 0 0.1" rpy="${pi/2} -${pi/2} 0" />
-      <parent link="stick_link1"/>
-      <child link="stick_link2"/>
+      <parent link="$(arg robot_name)_link1"/>
+      <child link="$(arg robot_name)_link2"/>
       <axis xyz="0 1 0"/>
       <limit acceleration="15" lower="-2.9671" effort="87" upper="2.9671" velocity="2.5"/>
@@ -95,9 +96,9 @@
   </xacro:unless>
   <!--  Weight joint-->
-  <joint name="stick_joint2" type="revolute">
+  <joint name="$(arg robot_name)_joint2" type="revolute">
     <safety_controller k_position="100.0" k_velocity="40.0" soft_lower_limit="-2.8973" soft_upper_limit="2.8973"/>
     <origin xyz="0 0 0.1" rpy="${pi/2} 0 0"/>
-    <parent link="stick_link2"/>
-    <child link="stick_link3"/>
+    <parent link="$(arg robot_name)_link2"/>
+    <child link="$(arg robot_name)_link3"/>
     <axis xyz="0 0 1"/>
     <limit acceleration="15" lower="-2.9671" effort="87" upper="2.9671" velocity="2.5"/>
@@ -105,27 +106,27 @@
   </joint>
   <!--Create hardware interfaces-->
-  <gazebo reference="stick_joint1">
+  <gazebo reference="$(arg robot_name)_joint1">
     <!-- Needed for ODE to output external wrenches on joints -->
     <provideFeedback>true</provideFeedback>
   </gazebo>
-  <gazebo reference="stick_joint2">
+  <gazebo reference="$(arg robot_name)_joint2">
     <!-- Needed for ODE to output external wrenches on joints -->
     <provideFeedback>true</provideFeedback>
   </gazebo>
-  <transmission name="stick_joint1_transmission">
+  <transmission name="$(arg robot_name)_joint1_transmission">
     <type>transmission_interface/SimpleTransmission</type>
-    <joint name="stick_joint1">
+    <joint name="$(arg robot_name)_joint1">
       <hardwareInterface>hardware_interface/EffortJointInterface</hardwareInterface>
     </joint>
-    <actuator name="stick_joint1_motor">
+    <actuator name="$(arg robot_name)_joint1_motor">
       <hardwareInterface>hardware_interface/EffortJointInterface</hardwareInterface>
     </actuator>
   </transmission>
-  <transmission name="stick_joint2_transmission">
+  <transmission name="$(arg robot_name)_joint2_transmission">
     <type>transmission_interface/SimpleTransmission</type>
-    <joint name="stick_joint2">
+    <joint name="$(arg robot_name)_joint2">
       <hardwareInterface>hardware_interface/EffortJointInterface</hardwareInterface>
     </joint>
-    <actuator name="stick_joint2_motor">
+    <actuator name="$(arg robot_name)_joint2_motor">
       <hardwareInterface>hardware_interface/EffortJointInterface</hardwareInterface>
     </actuator>

Commit message: feat: align stick orientations with franka_ros example

File: gazebo_torque_calculation_bug/stick_description/stick.urdf.xacro (robot description, xacro)
@@ -76,5 +76,5 @@
     <joint name="$(arg robot_name)_joint1" type="revolute">
       <safety_controller k_position="100.0" k_velocity="40.0" soft_lower_limit="-2.8973" soft_upper_limit="2.8973"/>
-      <origin xyz="0 0 0.1" rpy="${pi/2} -${pi/2} 0" />
+      <origin xyz="0 0 0.1" rpy="${pi/2} 0 0"/>
       <parent link="$(arg robot_name)_link1"/>
       <child link="$(arg robot_name)_link2"/>
@@ -87,5 +87,5 @@
     <joint name="$(arg robot_name)_joint1" type="revolute">
       <safety_controller k_position="100.0" k_velocity="40.0" soft_lower_limit="-2.8973" soft_upper_limit="2.8973"/>
-      <origin xyz="0 0 0.1" rpy="${pi/2} -${pi/2} 0" />
+      <origin xyz="0 0 0.1" rpy="0 0 0"/>
       <parent link="$(arg robot_name)_link1"/>
       <child link="$(arg robot_name)_link2"/>
