Commit message: feat: add panda joint positions

File: gazebo_torque_calculation_bug/stick_description/stick_long.urdf.xacro (robot description, xacro)
@@ -178,5 +178,5 @@
   <joint name="$(arg robot_name)_joint2" type="revolute">
     <safety_controller k_position="100.0" k_velocity="40.0" soft_lower_limit="-2.8973" soft_upper_limit="2.8973"/>
-    <origin xyz="0 0 0.1" rpy="0 0 0"/>
+    <origin xyz="0 0 0.1" rpy="${-pi/2} 0 0"/>
     <parent link="$(arg robot_name)_link2"/>
     <child link="$(arg robot_name)_link3"/>
@@ -187,5 +187,5 @@
   <joint name="$(arg robot_name)_joint3" type="revolute">
     <safety_controller k_position="100.0" k_velocity="40.0" soft_lower_limit="-2.8973" soft_upper_limit="2.8973"/>
-    <origin xyz="0 0 0.1" rpy="0 0 0"/>
+    <origin xyz="0 0 0.1" rpy="${pi/2} 0 0"/>
     <parent link="$(arg robot_name)_link3"/>
     <child link="$(arg robot_name)_link4"/>
@@ -196,5 +196,5 @@
   <joint name="$(arg robot_name)_joint4" type="revolute">
     <safety_controller k_position="100.0" k_velocity="40.0" soft_lower_limit="-2.8973" soft_upper_limit="2.8973"/>
-    <origin xyz="0 0 0.1" rpy="0 0 0"/>
+    <origin xyz="0 0 0.1" rpy="${pi/2} 0 0"/>
     <parent link="$(arg robot_name)_link4"/>
     <child link="$(arg robot_name)_link5"/>
@@ -205,5 +205,5 @@
   <joint name="$(arg robot_name)_joint5" type="revolute">
     <safety_controller k_position="100.0" k_velocity="40.0" soft_lower_limit="-2.8973" soft_upper_limit="2.8973"/>
-    <origin xyz="0 0 0.1" rpy="0 0 0"/>
+    <origin xyz="0 0 0.1" rpy="${-pi/2} 0 0"/>
     <parent link="$(arg robot_name)_link5"/>
     <child link="$(arg robot_name)_link6"/>
@@ -212,28 +212,13 @@
     <dynamics D="1" K="7000" mu_coulomb="0" mu_viscous="16" damping="0.003" friction="0.0"/>
   </joint>
-  <!--  Problem joint-->
-  <xacro:if value="$(arg rotated)">    <!--With rotation-->
-    <joint name="$(arg robot_name)_joint6" type="revolute">
-      <safety_controller k_position="100.0" k_velocity="40.0" soft_lower_limit="-2.8973" soft_upper_limit="2.8973"/>
-      <origin xyz="0 0 0.1" rpy="${pi/2} 0 0"/>
-      <parent link="$(arg robot_name)_link6"/>
-      <child link="$(arg robot_name)_link7"/>
-      <axis xyz="0 0 1"/>
-      <limit acceleration="15" lower="-2.9671" effort="87" upper="2.9671" velocity="2.5"/>
-      <dynamics D="1" K="7000" mu_coulomb="0" mu_viscous="16" damping="0.003" friction="0.0"/>
-    </joint>
-  </xacro:if>
-  <xacro:unless value="$(arg rotated)">
-    <joint name="$(arg robot_name)_joint6" type="revolute">
-      <safety_controller k_position="100.0" k_velocity="40.0" soft_lower_limit="-2.8973" soft_upper_limit="2.8973"/>
-      <origin xyz="0 0 0.1" rpy="0 0 0"/>
-      <parent link="$(arg robot_name)_link6"/>
-      <child link="$(arg robot_name)_link7"/>
-      <axis xyz="0 1 0"/>
-      <limit acceleration="15" lower="-2.9671" effort="87" upper="2.9671" velocity="2.5"/>
-      <dynamics D="1" K="7000" mu_coulomb="0" mu_viscous="16" damping="0.003" friction="0.0"/>
-    </joint>
-  </xacro:unless>
-  <!--  Weight joint-->
+  <joint name="$(arg robot_name)_joint6" type="revolute">
+    <safety_controller k_position="100.0" k_velocity="40.0" soft_lower_limit="-2.8973" soft_upper_limit="2.8973"/>
+    <origin xyz="0 0 0.1" rpy="${pi/2} 0 0"/>
+    <parent link="$(arg robot_name)_link6"/>
+    <child link="$(arg robot_name)_link7"/>
+    <axis xyz="0 0 1"/>
+    <limit acceleration="15" lower="-2.9671" effort="87" upper="2.9671" velocity="2.5"/>
+    <dynamics D="1" K="7000" mu_coulomb="0" mu_viscous="16" damping="0.003" friction="0.0"/>
+  </joint>
   <joint name="$(arg robot_name)_joint7" type="revolute">
     <safety_controller k_position="100.0" k_velocity="40.0" soft_lower_limit="-2.8973" soft_upper_limit="2.8973"/>

Commit message: feat: add joint lenghts/positions

File: gazebo_torque_calculation_bug/stick_description/stick_long.urdf.xacro (robot description, xacro)
@@ -169,5 +169,5 @@
   <joint name="$(arg robot_name)_joint1" type="revolute">
     <safety_controller k_position="100.0" k_velocity="40.0" soft_lower_limit="-2.8973" soft_upper_limit="2.8973"/>
-    <origin xyz="0 0 0.1" rpy="0 0 0"/>
+    <origin xyz="0 0 0.333" rpy="0 0 0"/>
     <parent link="$(arg robot_name)_link1"/>
     <child link="$(arg robot_name)_link2"/>
@@ -178,5 +178,5 @@
   <joint name="$(arg robot_name)_joint2" type="revolute">
     <safety_controller k_position="100.0" k_velocity="40.0" soft_lower_limit="-2.8973" soft_upper_limit="2.8973"/>
-    <origin xyz="0 0 0.1" rpy="${-pi/2} 0 0"/>
+    <origin xyz="0 0 0" rpy="${-pi/2} 0 0"/>
     <parent link="$(arg robot_name)_link2"/>
     <child link="$(arg robot_name)_link3"/>
@@ -187,5 +187,5 @@
   <joint name="$(arg robot_name)_joint3" type="revolute">
     <safety_controller k_position="100.0" k_velocity="40.0" soft_lower_limit="-2.8973" soft_upper_limit="2.8973"/>
-    <origin xyz="0 0 0.1" rpy="${pi/2} 0 0"/>
+    <origin xyz="0 -0.316 0" rpy="${pi/2} 0 0"/>
     <parent link="$(arg robot_name)_link3"/>
     <child link="$(arg robot_name)_link4"/>
@@ -196,5 +196,5 @@
   <joint name="$(arg robot_name)_joint4" type="revolute">
     <safety_controller k_position="100.0" k_velocity="40.0" soft_lower_limit="-2.8973" soft_upper_limit="2.8973"/>
-    <origin xyz="0 0 0.1" rpy="${pi/2} 0 0"/>
+    <origin xyz="0.0825 0 0" rpy="${pi/2} 0 0"/>
     <parent link="$(arg robot_name)_link4"/>
     <child link="$(arg robot_name)_link5"/>
@@ -205,5 +205,5 @@
   <joint name="$(arg robot_name)_joint5" type="revolute">
     <safety_controller k_position="100.0" k_velocity="40.0" soft_lower_limit="-2.8973" soft_upper_limit="2.8973"/>
-    <origin xyz="0 0 0.1" rpy="${-pi/2} 0 0"/>
+    <origin xyz="-0.0825 0.384 0" rpy="${-pi/2} 0 0"/>
     <parent link="$(arg robot_name)_link5"/>
     <child link="$(arg robot_name)_link6"/>
@@ -214,5 +214,5 @@
   <joint name="$(arg robot_name)_joint6" type="revolute">
     <safety_controller k_position="100.0" k_velocity="40.0" soft_lower_limit="-2.8973" soft_upper_limit="2.8973"/>
-    <origin xyz="0 0 0.1" rpy="${pi/2} 0 0"/>
+    <origin xyz="0 0 0" rpy="${pi/2} 0 0"/>
     <parent link="$(arg robot_name)_link6"/>
     <child link="$(arg robot_name)_link7"/>
@@ -223,5 +223,5 @@
   <joint name="$(arg robot_name)_joint7" type="revolute">
     <safety_controller k_position="100.0" k_velocity="40.0" soft_lower_limit="-2.8973" soft_upper_limit="2.8973"/>
-    <origin xyz="0 0 0.1" rpy="${pi/2} 0 0"/>
+    <origin xyz="0.088 0 0" rpy="${pi/2} 0 0"/>
     <parent link="$(arg robot_name)_link7"/>
     <child link="$(arg robot_name)_link8"/>

Commit message: feat: add panda meshes

File: gazebo_torque_calculation_bug/stick_description/stick_long.urdf.xacro (robot description, xacro)
@@ -16,13 +16,13 @@
   <link name="$(arg robot_name)_link1">
     <visual>
-      <origin xyz="0 0 0.05" />
-      <geometry>
-        <box size="0.02 0.02 0.08" />
-      </geometry>
-    </visual>
-    <collision>
-      <origin xyz="0 0 0.05" />
-      <geometry>
-        <box size="0.02 0.02 0.08" />
+      <origin rpy="0 0 0" xyz="0 0 0"/>
+      <geometry>
+        <mesh filename="package://franka_description/meshes/visual/link0.dae"/>
+      </geometry>
+    </visual>
+    <collision>
+    <origin rpy="0 0 0" xyz="0 0 0"/>
+      <geometry>
+        <mesh filename="package://franka_description/meshes/collision/link0.stl"/>
       </geometry>
     </collision>
@@ -35,13 +35,13 @@
   <link name="$(arg robot_name)_link2">
     <visual>
-      <origin xyz="0 0 0.05" />
-      <geometry>
-        <box size="0.02 0.02 0.08" />
-      </geometry>
-    </visual>
-    <collision>
-      <origin xyz="0 0 0.05" />
-      <geometry>
-        <box size="0.02 0.02 0.08" />
+      <origin rpy="0 0 0" xyz="0 0 0"/>
+      <geometry>
+        <mesh filename="package://franka_description/meshes/visual/link1.dae"/>
+      </geometry>
+    </visual>
+    <collision>
+      <origin rpy="0 0 0" xyz="0 0 0"/>
+      <geometry>
+        <mesh filename="package://franka_description/meshes/collision/link1.stl"/>
       </geometry>
     </collision>
@@ -54,13 +54,13 @@
   <link name="$(arg robot_name)_link3">
     <visual>
-      <origin xyz="0 0 0.05" />
-      <geometry>
-        <box size="0.02 0.02 0.08" />
-      </geometry>
-    </visual>
-    <collision>
-      <origin xyz="0 0 0.05" />
-      <geometry>
-        <box size="0.02 0.02 0.08" />
+      <origin rpy="0 0 0" xyz="0 0 0"/>
+      <geometry>
+        <mesh filename="package://franka_description/meshes/visual/link2.dae"/>
+      </geometry>
+    </visual>
+    <collision>
+      <origin rpy="0 0 0" xyz="0 0 0"/>
+      <geometry>
+        <mesh filename="package://franka_description/meshes/collision/link2.stl"/>
       </geometry>
     </collision>
@@ -73,13 +73,13 @@
   <link name="$(arg robot_name)_link4">
     <visual>
-      <origin xyz="0 0 0.05" />
-      <geometry>
-        <box size="0.02 0.02 0.08" />
-      </geometry>
-    </visual>
-    <collision>
-      <origin xyz="0 0 0.05" />
-      <geometry>
-        <box size="0.02 0.02 0.08" />
+      <origin rpy="0 0 0" xyz="0 0 0"/>
+      <geometry>
+        <mesh filename="package://franka_description/meshes/visual/link3.dae"/>
+      </geometry>
+    </visual>
+    <collision>
+      <origin rpy="0 0 0" xyz="0 0 0"/>
+      <geometry>
+        <mesh filename="package://franka_description/meshes/collision/link3.stl"/>
       </geometry>
     </collision>
@@ -92,13 +92,13 @@
   <link name="$(arg robot_name)_link5">
     <visual>
-      <origin xyz="0 0 0.05" />
-      <geometry>
-        <box size="0.02 0.02 0.08" />
-      </geometry>
-    </visual>
-    <collision>
-      <origin xyz="0 0 0.05" />
-      <geometry>
-        <box size="0.02 0.02 0.08" />
+      <origin rpy="0 0 0" xyz="0 0 0"/>
+      <geometry>
+        <mesh filename="package://franka_description/meshes/visual/link4.dae"/>
+      </geometry>
+    </visual>
+    <collision>
+      <origin rpy="0 0 0" xyz="0 0 0"/>
+      <geometry>
+        <mesh filename="package://franka_description/meshes/collision/link4.stl"/>
       </geometry>
     </collision>
@@ -111,13 +111,13 @@
   <link name="$(arg robot_name)_link6">
     <visual>
-      <origin xyz="0 0 0.05" />
-      <geometry>
-        <box size="0.02 0.02 0.08" />
-      </geometry>
-    </visual>
-    <collision>
-      <origin xyz="0 0 0.05" />
-      <geometry>
-        <box size="0.02 0.02 0.08" />
+      <origin rpy="0 0 0" xyz="0 0 0"/>
+      <geometry>
+        <mesh filename="package://franka_description/meshes/visual/link5.dae"/>
+      </geometry>
+    </visual>
+    <collision>
+      <origin rpy="0 0 0" xyz="0 0 0"/>
+      <geometry>
+        <mesh filename="package://franka_description/meshes/collision/link5.stl"/>
       </geometry>
     </collision>
@@ -130,13 +130,13 @@
   <link name="$(arg robot_name)_link7">
     <visual>
-      <origin xyz="0 0 0.05" />
-      <geometry>
-        <box size="0.02 0.02 0.08" />
-      </geometry>
-    </visual>
-    <collision>
-      <origin xyz="0 0 0.05" />
-      <geometry>
-        <box size="0.02 0.02 0.08" />
+      <origin rpy="0 0 0" xyz="0 0 0"/>
+      <geometry>
+        <mesh filename="package://franka_description/meshes/visual/link6.dae"/>
+      </geometry>
+    </visual>
+    <collision>
+      <origin rpy="0 0 0" xyz="0 0 0"/>
+      <geometry>
+        <mesh filename="package://franka_description/meshes/collision/link6.stl"/>
       </geometry>
     </collision>
@@ -149,13 +149,13 @@
   <link name="$(arg robot_name)_link8">
     <visual>
-      <origin xyz="0 0 0.05" />
-      <geometry>
-        <box size="0.02 0.02 0.08" />
-      </geometry>
-    </visual>
-    <collision>
-      <origin xyz="0 0 0.05" />
-      <geometry>
-        <box size="0.02 0.02 0.08" />
+      <origin rpy="0 0 0" xyz="0 0 0"/>
+      <geometry>
+        <mesh filename="package://franka_description/meshes/visual/link7.dae"/>
+      </geometry>
+    </visual>
+    <collision>
+      <origin rpy="0 0 0" xyz="0 0 0"/>
+      <geometry>
+        <mesh filename="package://franka_description/meshes/collision/link7.stl"/>
       </geometry>
     </collision>

Commit message: feat: add center of mass position

File: gazebo_torque_calculation_bug/stick_description/stick_long.urdf.xacro (robot description, xacro)
@@ -28,5 +28,5 @@
     </collision>
     <inertial>
-      <origin xyz="0 0 0.05" />
+      <origin rpy="0 0 0" xyz="-0.041018 -0.00014 0.049974"/>
       <mass value="${0.5*10./9.80}" />
       <inertia ixx="0.1" iyy="0.1" izz="0.1" ixy="0" ixz="0" iyz="0" />
@@ -47,5 +47,5 @@
     </collision>
     <inertial>
-      <origin xyz="0 0 0.05" />
+      <origin rpy="0 0 0" xyz="0.003875 0.002081 -0.04762"/>
       <mass value="${0.5*10./9.80}" />
       <inertia ixx="0.1" iyy="0.1" izz="0.1" ixy="0" ixz="0" iyz="0" />
@@ -66,5 +66,5 @@
     </collision>
     <inertial>
-      <origin xyz="0 0 0.05" />
+      <origin rpy="0 0 0" xyz=" -0.003141 -0.02872  0.003495"/>
       <mass value="${0.5*10./9.80}" />
       <inertia ixx="0.1" iyy="0.1" izz="0.1" ixy="0" ixz="0" iyz="0" />
@@ -85,5 +85,5 @@
     </collision>
     <inertial>
-      <origin xyz="0 0 0.05" />
+      <origin rpy="0 0 0" xyz="2.7518e-02 3.9252e-02 -6.6502e-02"/>
       <mass value="${0.5*10./9.80}" />
       <inertia ixx="0.1" iyy="0.1" izz="0.1" ixy="0" ixz="0" iyz="0" />
@@ -104,5 +104,5 @@
     </collision>
     <inertial>
-      <origin xyz="0 0 0.05" />
+      <origin rpy="0 0 0" xyz="-5.317e-02 1.04419e-01 2.7454e-02"/>
       <mass value="${0.5*10./9.80}" />
       <inertia ixx="0.1" iyy="0.1" izz="0.1" ixy="0" ixz="0" iyz="0" />
@@ -123,5 +123,5 @@
     </collision>
     <inertial>
-      <origin xyz="0 0 0.05" />
+      <origin rpy="0 0 0" xyz="-1.1953e-02 4.1065e-02 -3.8437e-02"/>
       <mass value="${0.5*10./9.80}" />
       <inertia ixx="0.1" iyy="0.1" izz="0.1" ixy="0" ixz="0" iyz="0" />
@@ -142,5 +142,5 @@
     </collision>
     <inertial>
-      <origin xyz="0 0 0.05" />
+      <origin rpy="0 0 0" xyz="6.0149e-02 -1.4117e-02 -1.0517e-02"/>
       <mass value="${0.5*10./9.80}" />
       <inertia ixx="0.1" iyy="0.1" izz="0.1" ixy="0" ixz="0" iyz="0" />
@@ -161,5 +161,5 @@
     </collision>
     <inertial>
-      <origin xyz="0 0 0.05" />
+      <origin rpy="0 0 0" xyz="1.0517e-02 -4.252e-03 6.1597e-02"/>
       <mass value="${0.5*10./9.80}" />
       <inertia ixx="0.1" iyy="0.1" izz="0.1" ixy="0" ixz="0" iyz="0" />

Commit message: feat: add actual robot mass

File: gazebo_torque_calculation_bug/stick_description/stick_long.urdf.xacro (robot description, xacro)
@@ -29,5 +29,5 @@
     <inertial>
       <origin rpy="0 0 0" xyz="-0.041018 -0.00014 0.049974"/>
-      <mass value="${0.5*10./9.80}" />
+      <mass value="0.629769"/>
       <inertia ixx="0.1" iyy="0.1" izz="0.1" ixy="0" ixz="0" iyz="0" />
     </inertial>
@@ -48,5 +48,5 @@
     <inertial>
       <origin rpy="0 0 0" xyz="0.003875 0.002081 -0.04762"/>
-      <mass value="${0.5*10./9.80}" />
+      <mass value="4.970684"/>
       <inertia ixx="0.1" iyy="0.1" izz="0.1" ixy="0" ixz="0" iyz="0" />
     </inertial>
@@ -67,5 +67,5 @@
     <inertial>
       <origin rpy="0 0 0" xyz=" -0.003141 -0.02872  0.003495"/>
-      <mass value="${0.5*10./9.80}" />
+      <mass value="0.646926"/>
       <inertia ixx="0.1" iyy="0.1" izz="0.1" ixy="0" ixz="0" iyz="0" />
     </inertial>
@@ -86,5 +86,5 @@
     <inertial>
       <origin rpy="0 0 0" xyz="2.7518e-02 3.9252e-02 -6.6502e-02"/>
-      <mass value="${0.5*10./9.80}" />
+      <mass value="3.228604"/>
       <inertia ixx="0.1" iyy="0.1" izz="0.1" ixy="0" ixz="0" iyz="0" />
     </inertial>
@@ -105,5 +105,5 @@
     <inertial>
       <origin rpy="0 0 0" xyz="-5.317e-02 1.04419e-01 2.7454e-02"/>
-      <mass value="${0.5*10./9.80}" />
+      <mass value="3.587895"/>
       <inertia ixx="0.1" iyy="0.1" izz="0.1" ixy="0" ixz="0" iyz="0" />
     </inertial>
@@ -124,5 +124,5 @@
     <inertial>
       <origin rpy="0 0 0" xyz="-1.1953e-02 4.1065e-02 -3.8437e-02"/>
-      <mass value="${0.5*10./9.80}" />
+      <mass value="1.225946"/>
       <inertia ixx="0.1" iyy="0.1" izz="0.1" ixy="0" ixz="0" iyz="0" />
     </inertial>
@@ -143,5 +143,5 @@
     <inertial>
       <origin rpy="0 0 0" xyz="6.0149e-02 -1.4117e-02 -1.0517e-02"/>
-      <mass value="${0.5*10./9.80}" />
+      <mass value="1.666555"/>
       <inertia ixx="0.1" iyy="0.1" izz="0.1" ixy="0" ixz="0" iyz="0" />
     </inertial>
@@ -162,5 +162,5 @@
     <inertial>
       <origin rpy="0 0 0" xyz="1.0517e-02 -4.252e-03 6.1597e-02"/>
-      <mass value="${0.5*10./9.80}" />
+      <mass value="7.35522e-01"/>
       <inertia ixx="0.1" iyy="0.1" izz="0.1" ixy="0" ixz="0" iyz="0" />
     </inertial>
