Commit message: feat: add moment of inertia

File: gazebo_torque_calculation_bug/stick_description/stick_long.urdf.xacro (robot description, xacro)
@@ -6,4 +6,5 @@
   <xacro:arg name="rotated" default="false" />
   <xacro:arg name="robot_name" default="stick" />
+  <xacro:arg name="safety_controller" default="true" />
   <!--Gazebo requires a joint to a link called "world" for statically mounted robots-->
   <link name="world" />
@@ -30,5 +31,7 @@
       <origin rpy="0 0 0" xyz="-0.041018 -0.00014 0.049974"/>
       <mass value="0.629769"/>
-      <inertia ixx="0.1" iyy="0.1" izz="0.1" ixy="0" ixz="0" iyz="0" />
+      <inertia ixx="0.00315" ixy="8.2904E-07" ixz="0.00015"
+                              iyy="0.00388"    iyz="8.2299E-06"
+                                              izz="0.004285" />
     </inertial>
   </link>
@@ -49,5 +52,8 @@
       <origin rpy="0 0 0" xyz="0.003875 0.002081 -0.04762"/>
       <mass value="4.970684"/>
-      <inertia ixx="0.1" iyy="0.1" izz="0.1" ixy="0" ixz="0" iyz="0" />
+      <mass value="4.970684"/>
+      <inertia ixx="0.70337" ixy="-0.00013900" ixz="0.0067720"
+                             iyy="0.70661"     iyz="0.019169"
+                                               izz="0.0091170" />
     </inertial>
   </link>
@@ -68,5 +74,7 @@
       <origin rpy="0 0 0" xyz=" -0.003141 -0.02872  0.003495"/>
       <mass value="0.646926"/>
-      <inertia ixx="0.1" iyy="0.1" izz="0.1" ixy="0" ixz="0" iyz="0" />
+      <inertia ixx="0.0079620" ixy="-3.9250e-3" ixz="1.0254e-02"
+                               iyy="2.8110e-02" iyz="7.0400e-04"
+                                                izz="2.5995e-02" />
     </inertial>
   </link>
@@ -87,5 +95,7 @@
       <origin rpy="0 0 0" xyz="2.7518e-02 3.9252e-02 -6.6502e-02"/>
       <mass value="3.228604"/>
-      <inertia ixx="0.1" iyy="0.1" izz="0.1" ixy="0" ixz="0" iyz="0" />
+      <inertia ixx="3.7242e-02" ixy="-4.7610e-03" ixz="-1.1396e-02"
+                                iyy="3.6155e-02"  iyz="-1.2805e-02"
+                                                  izz="1.0830e-02" />
     </inertial>
   </link>
@@ -106,5 +116,7 @@
       <origin rpy="0 0 0" xyz="-5.317e-02 1.04419e-01 2.7454e-02"/>
       <mass value="3.587895"/>
-      <inertia ixx="0.1" iyy="0.1" izz="0.1" ixy="0" ixz="0" iyz="0" />
+      <inertia ixx="2.5853e-02" ixy="7.7960e-03" ixz="-1.3320e-03"
+                                iyy="1.9552e-02" iyz="8.6410e-03"
+                                                  izz="2.8323e-02" />
     </inertial>
   </link>
@@ -125,5 +137,7 @@
       <origin rpy="0 0 0" xyz="-1.1953e-02 4.1065e-02 -3.8437e-02"/>
       <mass value="1.225946"/>
-      <inertia ixx="0.1" iyy="0.1" izz="0.1" ixy="0" ixz="0" iyz="0" />
+      <inertia ixx="3.5549e-02" ixy="-2.1170e-03" ixz="-4.0370e-03"
+                                iyy="2.9474e-02"  iyz="2.2900e-04"
+                                                  izz="8.6270e-03" />
     </inertial>
   </link>
@@ -144,5 +158,7 @@
       <origin rpy="0 0 0" xyz="6.0149e-02 -1.4117e-02 -1.0517e-02"/>
       <mass value="1.666555"/>
-      <inertia ixx="0.1" iyy="0.1" izz="0.1" ixy="0" ixz="0" iyz="0" />
+      <inertia ixx="1.9640e-03" ixy="1.0900e-04" ixz="-1.1580e-03"
+                                iyy="4.3540e-03" iyz="3.4100e-04"
+                                                  izz="5.4330e-03" />
     </inertial>
   </link>
@@ -163,10 +179,14 @@
       <origin rpy="0 0 0" xyz="1.0517e-02 -4.252e-03 6.1597e-02"/>
       <mass value="7.35522e-01"/>
-      <inertia ixx="0.1" iyy="0.1" izz="0.1" ixy="0" ixz="0" iyz="0" />
+      <inertia ixx="1.2516e-02" ixy="-4.2800e-04" ixz="-1.1960e-03"
+                                iyy="1.0027e-02"  iyz="-7.4100e-04"
+                                                  izz="4.8150e-03"/>
     </inertial>
   </link>
   <!--Create stick joints-->
   <joint name="$(arg robot_name)_joint1" type="revolute">
-    <safety_controller k_position="100.0" k_velocity="40.0" soft_lower_limit="-2.8973" soft_upper_limit="2.8973"/>
+    <xacro:if value="$(arg safety_controller)">
+      <safety_controller k_position="100.0" k_velocity="40.0" soft_lower_limit="-2.8973" soft_upper_limit="2.8973"/>
+    </xacro:if>
     <origin xyz="0 0 0.333" rpy="0 0 0"/>
     <parent link="$(arg robot_name)_link1"/>
@@ -177,5 +197,7 @@
   </joint>
   <joint name="$(arg robot_name)_joint2" type="revolute">
-    <safety_controller k_position="100.0" k_velocity="40.0" soft_lower_limit="-2.8973" soft_upper_limit="2.8973"/>
+    <xacro:if value="$(arg safety_controller)">
+      <safety_controller k_position="100.0" k_velocity="40.0" soft_lower_limit="-1.7628" soft_upper_limit="1.7628"/>
+    </xacro:if>
     <origin xyz="0 0 0" rpy="${-pi/2} 0 0"/>
     <parent link="$(arg robot_name)_link2"/>
@@ -186,5 +208,7 @@
   </joint>
   <joint name="$(arg robot_name)_joint3" type="revolute">
-    <safety_controller k_position="100.0" k_velocity="40.0" soft_lower_limit="-2.8973" soft_upper_limit="2.8973"/>
+    <xacro:if value="$(arg safety_controller)">
+      <safety_controller k_position="100.0" k_velocity="40.0" soft_lower_limit="-2.8973" soft_upper_limit="2.8973"/>
+    </xacro:if>
     <origin xyz="0 -0.316 0" rpy="${pi/2} 0 0"/>
     <parent link="$(arg robot_name)_link3"/>
@@ -195,5 +219,7 @@
   </joint>
   <joint name="$(arg robot_name)_joint4" type="revolute">
-    <safety_controller k_position="100.0" k_velocity="40.0" soft_lower_limit="-2.8973" soft_upper_limit="2.8973"/>
+    <xacro:if value="$(arg safety_controller)">
+      <safety_controller k_position="100.0" k_velocity="40.0" soft_lower_limit="-3.0718" soft_upper_limit="-0.0698"/>
+    </xacro:if>
     <origin xyz="0.0825 0 0" rpy="${pi/2} 0 0"/>
     <parent link="$(arg robot_name)_link4"/>
@@ -204,5 +230,7 @@
   </joint>
   <joint name="$(arg robot_name)_joint5" type="revolute">
-    <safety_controller k_position="100.0" k_velocity="40.0" soft_lower_limit="-2.8973" soft_upper_limit="2.8973"/>
+    <xacro:if value="$(arg safety_controller)">
+      <safety_controller k_position="100.0" k_velocity="40.0" soft_lower_limit="-2.8973" soft_upper_limit="2.8973"/>
+    </xacro:if>
     <origin xyz="-0.0825 0.384 0" rpy="${-pi/2} 0 0"/>
     <parent link="$(arg robot_name)_link5"/>
@@ -213,5 +241,7 @@
   </joint>
   <joint name="$(arg robot_name)_joint6" type="revolute">
-    <safety_controller k_position="100.0" k_velocity="40.0" soft_lower_limit="-2.8973" soft_upper_limit="2.8973"/>
+    <xacro:if value="$(arg safety_controller)">
+      <safety_controller k_position="100.0" k_velocity="40.0" soft_lower_limit="-0.0175" soft_upper_limit="3.7525"/>
+    </xacro:if>
     <origin xyz="0 0 0" rpy="${pi/2} 0 0"/>
     <parent link="$(arg robot_name)_link6"/>
@@ -222,5 +252,7 @@
   </joint>
   <joint name="$(arg robot_name)_joint7" type="revolute">
-    <safety_controller k_position="100.0" k_velocity="40.0" soft_lower_limit="-2.8973" soft_upper_limit="2.8973"/>
+    <xacro:if value="$(arg safety_controller)">
+      <safety_controller k_position="100.0" k_velocity="40.0" soft_lower_limit="-2.8973" soft_upper_limit="2.8973"/>
+    </xacro:if>
     <origin xyz="0.088 0 0" rpy="${pi/2} 0 0"/>
     <parent link="$(arg robot_name)_link7"/>

Commit message: feat: add joint properties

File: gazebo_torque_calculation_bug/stick_description/stick_long.urdf.xacro (robot description, xacro)
@@ -204,5 +204,5 @@
     <child link="$(arg robot_name)_link3"/>
     <axis xyz="0 0 1"/>
-    <limit acceleration="15" lower="-2.9671" effort="87" upper="2.9671" velocity="2.5"/>
+    <limit acceleration="7.5" lower="-1.8326" effort="87" upper="1.8326" velocity="2.5"/>
     <dynamics D="1" K="7000" mu_coulomb="0" mu_viscous="16" damping="0.003" friction="0.0"/>
   </joint>
@@ -215,5 +215,5 @@
     <child link="$(arg robot_name)_link4"/>
     <axis xyz="0 0 1"/>
-    <limit acceleration="15" lower="-2.9671" effort="87" upper="2.9671" velocity="2.5"/>
+    <limit acceleration="12.5" lower="-2.9671" effort="87" upper="2.9671" velocity="2.5"/>
     <dynamics D="1" K="7000" mu_coulomb="0" mu_viscous="16" damping="0.003" friction="0.0"/>
   </joint>
@@ -226,5 +226,5 @@
     <child link="$(arg robot_name)_link5"/>
     <axis xyz="0 0 1"/>
-    <limit acceleration="15" lower="-2.9671" effort="87" upper="2.9671" velocity="2.5"/>
+    <limit acceleration="12.5" lower="-3.1416" effort="87" upper="-0.4" velocity="2.5"/>
     <dynamics D="1" K="7000" mu_coulomb="0" mu_viscous="16" damping="0.003" friction="0.0"/>
   </joint>
@@ -237,5 +237,5 @@
     <child link="$(arg robot_name)_link6"/>
     <axis xyz="0 0 1"/>
-    <limit acceleration="15" lower="-2.9671" effort="87" upper="2.9671" velocity="2.5"/>
+    <limit acceleration="15" lower="-2.9671" effort="12" upper="2.9671" velocity="3"/>
     <dynamics D="1" K="7000" mu_coulomb="0" mu_viscous="16" damping="0.003" friction="0.0"/>
   </joint>
@@ -248,5 +248,5 @@
     <child link="$(arg robot_name)_link7"/>
     <axis xyz="0 0 1"/>
-    <limit acceleration="15" lower="-2.9671" effort="87" upper="2.9671" velocity="2.5"/>
+    <limit acceleration="20" lower="-0.0873" effort="12" upper="3.8223" velocity="3"/>
     <dynamics D="1" K="7000" mu_coulomb="0" mu_viscous="16" damping="0.003" friction="0.0"/>
   </joint>
@@ -259,5 +259,5 @@
     <child link="$(arg robot_name)_link8"/>
     <axis xyz="0 0 1"/>
-    <limit acceleration="15" lower="-2.9671" effort="87" upper="2.9671" velocity="2.5"/>
+    <limit acceleration="20" lower="-2.9671" effort="12" upper="2.9671" velocity="3"/>
     <dynamics D="1" K="7000" mu_coulomb="0" mu_viscous="16" damping="0.003" friction="0.0"/>
   </joint>
